Commit message: change the friction

File: urdf_models/models/blue_plate/model.urdf (robot description, URDF)
Before this commit: robot model.urdf, 1 links, 0 joints
Links:
- link baseLink: geometry collision mesh filename=collision.obj scale=0.5 0.5 0.5; visual mesh filename=textured.obj scale=0.5 0.5 0.5
